Commit message: fix: add petanque_ball frame to explorer tool

File: explorer_description/urdf/explorer.urdf.xacro (robot description, xacro)
@@ -65,4 +65,5 @@
   <link name="drink_small"/>
   <link name="drink_big"/>
+  <link name="petanque_ball"/>
   <joint name="joint-drink-small" type="fixed">
     <parent link="tool0"/>
@@ -76,4 +77,9 @@
     <!-- Lateral shift: 60mm in Y direction for big drinks -->
     <origin xyz="0 -0.045 0.045" rpy="0 0 0"/>
+  </joint>
+  <joint name="joint-petanque-ball" type="fixed">
+    <parent link="tool0"/>
+    <child link="petanque_ball"/>
+    <origin xyz="0.1 0 0" rpy="0 0 0"/>
   </joint>
   <xacro:gripper_pincette/>

Commit message: feat - petanque parameter

File: explorer_description/urdf/explorer.urdf.xacro (robot description, xacro)
@@ -20,5 +20,5 @@
     <parent link="world"/>
     <child link="base_link"/>
-    <origin xyz="0 0 0" rpy="0 0 0"/>
+    <origin xyz="0 0 1" rpy="0 0 0"/>
     <axis xyz="0 0 1"/>
   </joint>
@@ -65,4 +65,5 @@
   <link name="drink_small"/>
   <link name="drink_big"/>
+  <link name="petanque_ball"/>
   <joint name="joint-drink-small" type="fixed">
     <parent link="tool0"/>
@@ -76,4 +77,9 @@
     <!-- Lateral shift: 60mm in Y direction for big drinks -->
     <origin xyz="0 -0.045 0.045" rpy="0 0 0"/>
+  </joint>
+  <joint name="joint-petanque-ball" type="fixed">
+    <parent link="tool0"/>
+    <child link="petanque_ball"/>
+    <origin xyz="0.1 0 0" rpy="0 0 0"/>
   </joint>
   <xacro:gripper_pincette/>

File: explorer_description/urdf/explorer_joints.xacro (robot description, xacro)
@@ -12,5 +12,5 @@
         </command_interface>
         <state_interface name="position">
-          <param name="initial_value">0.0</param>
+          <param name="initial_value">-0.90</param>
         </state_interface>
         <state_interface name="velocity"/>
@@ -29,5 +29,5 @@
         </command_interface>
         <state_interface name="position">
-          <param name="initial_value">1.71</param>
+          <param name="initial_value">0.9</param>
         </state_interface>
         <state_interface name="velocity"/>
@@ -46,5 +46,5 @@
         </command_interface>
         <state_interface name="position">
-          <param name="initial_value">2.5</param>
+          <param name="initial_value">-0.4</param>
         </state_interface>
         <state_interface name="velocity"/>
@@ -80,5 +80,5 @@
         </command_interface>
         <state_interface name="position">
-          <param name="initial_value">-0.17</param>
+          <param name="initial_value">1.</param>
         </state_interface>
         <state_interface name="velocity"/>
@@ -97,5 +97,5 @@
         </command_interface>
         <state_interface name="position">
-          <param name="initial_value">0.0</param>
+          <param name="initial_value">-1.</param>
         </state_interface>
         <state_interface name="velocity"/>
